File: Design_IMX6QP/IMXDesign/CPU_DDR3.sch (KiCad schematic (older format))
At the start: 2 parts, among them U1 MCIMX6QP5EVT

Commit message: Update IMX6QP and IMX8MQ
Parts:
- added C153: 100nF, Capacitor_SMD:C_0402_1005Metric, symbol Device:C_Small
Connections:
- net GND: now also C153.2
- net DRAM_CAS renamed DRAM_CAS_B
- net DRAM_CS0 renamed DRAM_CS0_B
- net DRAM_RAS renamed DRAM_RAS_B
- net DRAM_SCS1: no longer names the net of U1.AD17 (DRAM_CS1)
- net DRAM_SDCKE1: no longer names the net of U1.AA11 (DRAM_SDCKE1)
- net DRAM_SDODT1: no longer names the net of U1.AB17 (DRAM_SDODT1)
- net DRAM_SDQS0 renamed DRAM_SDQS0+
- net DRAM_SDQS0_B renamed DRAM_SDQS0-
- net DRAM_SDQS1 renamed DRAM_SDQS1+
- net DRAM_SDQS1_B renamed DRAM_SDQS1-
- net DRAM_SDQS2 renamed DRAM_SDQS2+
- net DRAM_SDQS2_B renamed DRAM_SDQS2-
- net DRAM_SDQS3 renamed DRAM_SDQS3+
- net DRAM_SDQS3_B renamed DRAM_SDQS3-
- net DRAM_SDQS4 renamed DRAM_SDQS4+
- net DRAM_SDQS4_B renamed DRAM_SDQS4-
- net DRAM_SDQS5 renamed DRAM_SDQS5+
- net DRAM_SDQS5_B renamed DRAM_SDQS5-
- net DRAM_SDQS6 renamed DRAM_SDQS6+
- net DRAM_SDQS6_B renamed DRAM_SDQS6-
- net DRAM_SDQS7 renamed DRAM_SDQS7+
- net DRAM_SDQS7_B renamed DRAM_SDQS7-
- net DRAM_SDWE renamed DRAM_WE_B
- net DRAM_VREF renamed DDR_VREF
- net DDR_VREF: now also C153.1
- no-connect marks 0 -> 3
Other:
- moved on the sheet: R1, U1U
