File: Design_IMX6QP/IMXDesign/IMXDesign.sch (KiCad schematic (older format))
At the start: 1 part, among them U1 MCIMX6QP5EVT

Commit message: Update IMX6QP and IMX8MQ
Parts:
- removed unit 5 of U1
- removed unit 6 of U1
- removed unit 7 of U1
- removed unit 8 of U1
- removed unit 9 of U1
- removed unit 10 of U1
- removed unit 11 of U1
- removed unit 13 of U1
- removed unit 16 of U1
- removed unit 17 of U1
Other:
- moved on the sheet: U1B, U1C, U1D, U1L
