File: Design_IMX6QP/IMXDesign/MEM_DDR3.sch (KiCad schematic (older format))
At the start: 8 parts, among them U2 MT41K128M16JT-107_K, U3 MT41K128M16JT-107_K, U4 MT41K128M16JT-107_K, U5 MT41K128M16JT-107_K

Commit message: Update IMX6QP and IMX8MQ
Parts:
- removed U5: MT41K128M16JT-107_K, IMX6QP:BGA80P96C6X16_800X1400X110, symbol MT41K128M16JT-107_K:MT41K128M16JT-107_K
- added U5: MT41K128M16JT-107_K-MT41K128M16JT-107_K, IMX6QP:BGA80P96C6X16_800X1400X110, symbol IMXDesign-rescue:MT41K128M16JT-107_K-MT41K128M16JT-107_K
- U2, U3, U4: symbol MT41K128M16JT-107_K:MT41K128M16JT-107_K -> IMXDesign-rescue:MT41K128M16JT-107_K-MT41K128M16JT-107_K
Connections:
- net DDR_VREF: now also U5.H1 (VREFDQ), U5.M8 (VREFCA)
- net DRAM_A0: now also U5.N3 (A0)
- net DRAM_A1: now also U5.P7 (A1)
- net DRAM_A10: now also U5.L7 (A10/AP)
- net DRAM_A11: now also U5.R7 (A11)
- net DRAM_A12: now also U5.N7 (A12/~BC)
- net DRAM_A13: now also U5.T3 (A13)
- net DRAM_A14: now also U2.T7 (NC), U3.T7 (NC), U4.T7 (NC), U5.T7 (NC); no longer U3.M2 (BA0)
- net DRAM_A15: now also U2.M7 (NC), U3.M7 (NC), U4.M7 (NC), U5.M7 (NC); no longer U3.N8 (BA1)
- net DRAM_A2: now also U5.P3 (A2)
- net DRAM_A3: now also U5.N2 (A3)
- net DRAM_A4: now also U5.P8 (A4)
- net DRAM_A5: now also U5.P2 (A5)
- net DRAM_A6: now also U5.R8 (A6)
- net DRAM_A7: now also U5.R2 (A7)
- net DRAM_A8: now also U5.T8 (A8)
- net DRAM_A9: now also U5.R3 (A9)
- net DRAM_D1: now also U3.F8 (DQ3); no longer U3.F7 (DQ1)
- net DRAM_D10: now also U3.A2 (DQ13); no longer U3.C8 (DQ10)
- net DRAM_D11: now also U3.B8 (DQ14); no longer U3.C2 (DQ11)
- net DRAM_D12: now also U3.A3 (DQ15); no longer U3.A7 (DQ12)
- net DRAM_D13: now also U3.C2 (DQ11); no longer U3.A2 (DQ13)
- net DRAM_D14: now also U3.C3 (DQ9); no longer U3.B8 (DQ14)
- net DRAM_D15: now also U3.C8 (DQ10); no longer U3.A3 (DQ15)
- net DRAM_D3: now also U3.H3 (DQ4); no longer U3.F8 (DQ3)
- net DRAM_D4: now also U3.G2 (DQ6); no longer U3.H3 (DQ4)
- net DRAM_D6: now also U3.H7 (DQ7); no longer U3.G2 (DQ6)
- net DRAM_D7: now also U3.F7 (DQ1); no longer U3.H7 (DQ7)
- net DRAM_D9: now also U3.A7 (DQ12); no longer U3.C3 (DQ9)
- net DRAM_SDCLK_0+: now also U5.J7 (CK)
- net DRAM_SDCLK_0-: now also U5.K7 (~CK)
- net GND: now also U5.A9 (VSS), U5.B1 (VSSQ), U5.B3 (VSS), U5.B9 (VSSQ), U5.D1 (VSSQ), U5.D8 (VSSQ), U5.E1 (VSS), U5.E2 (VSSQ), U5.E8 (VSSQ), U5.F9 (VSSQ), U5.G1 (VSSQ), U5.G8 (VSS), U5.G9 (VSSQ), U5.J2 (VSS), U5.J8 (VSS), U5.M1 (VSS), U5.M9 (VSS), U5.P1 (VSS), U5.P9 (VSS), U5.T1 (VSS), U5.T9 (VSS)
- net at R5.1: now also U5.L8 (ZQ)
- net DRAM_D19: now reaches U2.A2 (DQ13)
- net DRAM_D23: now reaches U2.A3 (DQ15)
- net DRAM_D21: now reaches U2.A7 (DQ12)
- net DRAM_SDQS2-: now reaches U2.B7 (~UDQS)
- net DRAM_D20: now reaches U2.B8 (DQ14)
- net DRAM_D22: now reaches U2.C2 (DQ11)
- net DRAM_D18: now reaches U2.C3 (DQ9)
- net DRAM_SDQS2+: now reaches U2.C7 (UDQS)
- net DRAM_D17: now reaches U2.C8 (DQ10)
- net DRAM_DQM2: now reaches U2.D3 (UDM)
- net DRAM_D16: now reaches U2.D7 (DQ8)
- net DRAM_D24: now reaches U2.E3 (DQ0)
- net DRAM_DQM3: now reaches U2.E7 (LDM)
- net DRAM_D29: now reaches U2.F2 (DQ2)
- net DRAM_SDQS3+: now reaches U2.F3 (LDQS)
- net DRAM_D28: now reaches U2.F7 (DQ1)
- net DRAM_D27: now reaches U2.F8 (DQ3)
- net DRAM_D31: now reaches U2.G2 (DQ6)
- net DRAM_SDQS3-: now reaches U2.G3 (~LDQS)
- net DRAM_D25: now reaches U2.H3 (DQ4)
- net DRAM_D30: now reaches U2.H7 (DQ7)
- net DRAM_D26: now reaches U2.H8 (DQ5)
- net DRAM_RAS_B: now reaches U2.J3 (~RAS)
- net DRAM_RAS_B: now also U3.J3 (~RAS), U4.J3 (~RAS), U5.J3 (~RAS)
- net DRAM_SDODT0: now reaches U2.K1 (ODT)
- net DRAM_SDODT0: now also U3.K1 (ODT), U4.K1 (ODT), U5.K1 (ODT)
- net DRAM_CAS_B: now reaches U2.K3 (~CAS)
- net DRAM_CAS_B: now also U3.K3 (~CAS), U4.K3 (~CAS), U5.K3 (~CAS)
- net DRAM_SDCKE0: now reaches U2.K9 (CKE)
- net DRAM_SDCKE0: now also U3.K9 (CKE), U4.K9 (CKE), U5.K9 (CKE)
- net DRAM_CS0_B: now reaches U2.L2 (~CS)
- net DRAM_CS0_B: now also U3.L2 (~CS), U4.L2 (~CS), U5.L2 (~CS)
- net DRAM_SDWE_B: now reaches U2.L3 (~WE)
- net DRAM_SDWE_B: now also U3.L3 (~WE), U4.L3 (~WE), U5.L3 (~WE)
- net DRAM_SDBA2: now reaches U2.M2 (BA0)
- net DRAM_SDBA2: now also U3.M2 (BA0), U4.M2 (BA0), U5.M2 (BA0)
- net DRAM_SDBA0: now reaches U2.M3 (BA2)
- net DRAM_SDBA0: now also U3.M3 (BA2), U4.M3 (BA2), U5.M3 (BA2)
- net DRAM_SDBA1: now reaches U2.N8 (BA1)
- net DRAM_SDBA1: now also U3.N8 (BA1), U4.N8 (BA1), U5.N8 (BA1)
- net DRAM_D43: now reaches U4.A2 (DQ13)
- net DRAM_D41: now reaches U4.A3 (DQ15)
- net DRAM_D46: now reaches U4.A7 (DQ12)
- net DRAM_SDQS5-: now reaches U4.B7 (~UDQS)
- net DRAM_D42: now reaches U4.B8 (DQ14)
- net DRAM_D44: now reaches U4.C2 (DQ11)
- net DRAM_D45: now reaches U4.C3 (DQ9)
- net DRAM_SDQS5+: now reaches U4.C7 (UDQS)
- net DRAM_D47: now reaches U4.C8 (DQ10)
- net DRAM_DQM5: now reaches U4.D3 (UDM)
- net DRAM_D40: now reaches U4.D7 (DQ8)
- net DRAM_D32: now reaches U4.E3 (DQ0)
- net DRAM_DQM4: now reaches U4.E7 (LDM)
- net DRAM_D39: now reaches U4.F2 (DQ2)
- net DRAM_SDQS4+: now reaches U4.F3 (LDQS)
- net DRAM_D38: now reaches U4.F7 (DQ1)
- net DRAM_D35: now reaches U4.F8 (DQ3)
- net DRAM_D34: now reaches U4.G2 (DQ6)
- net DRAM_SDQS4-: now reaches U4.G3 (~LDQS)
- net DRAM_D37: now reaches U4.H3 (DQ4)
- net DRAM_D36: now reaches U4.H7 (DQ7)
- net DRAM_D33: now reaches U4.H8 (DQ5)
- net DRAM_SDQS1-: now reaches U3.B7 (~UDQS)
- net DRAM_SDQS1+: now reaches U3.C7 (UDQS)
- net DRAM_DQM1: now reaches U3.D3 (UDM)
- net DRAM_DQM0: now reaches U3.E7 (LDM)
- net DRAM_SDQS0+: now reaches U3.F3 (LDQS)
- net DRAM_SDQS0-: now reaches U3.G3 (~LDQS)
- net +1v5_DDR renamed VDD
- net VDD: now also U5.A1 (VDDQ), U5.A8 (VDDQ), U5.B2 (VDD), U5.C1 (VDDQ), U5.C9 (VDDQ), U5.D2 (VDDQ), U5.D9 (VDD), U5.E9 (VDDQ), U5.F1 (VDDQ), U5.G7 (VDD), U5.H2 (VDDQ), U5.H9 (VDDQ), U5.K2 (VDD), U5.K8 (VDD), U5.N1 (VDD), U5.N9 (VDD), U5.R1 (VDD), U5.R9 (VDD)
- new net DRAM_D48: U5.D7 (DQ8)
- new net DRAM_D49: U5.C8 (DQ10)
- new net DRAM_D50: U5.A3 (DQ15)
- new net DRAM_D51: U5.C3 (DQ9)
- new net DRAM_D52: U5.B8 (DQ14)
- new net DRAM_D53: U5.A7 (DQ12)
- new net DRAM_D54: U5.A2 (DQ13)
- new net DRAM_D55: U5.C2 (DQ11)
- new net DRAM_D56: U5.E3 (DQ0)
- new net DRAM_D57: U5.H7 (DQ7)
- new net DRAM_D58: U5.H3 (DQ4)
- new net DRAM_D59: U5.H8 (DQ5)
- new net DRAM_D60: U5.F8 (DQ3)
- new net DRAM_D61: U5.F2 (DQ2)
- new net DRAM_D62: U5.F7 (DQ1)
- new net DRAM_D63: U5.G2 (DQ6)
- new net DRAM_DQM6: U5.D3 (UDM)
- new net DRAM_DQM7: U5.E7 (LDM)
- new net DRAM_SDQS6+: U5.C7 (UDQS)
- new net DRAM_SDQS6-: U5.B7 (~UDQS)
- new net DRAM_SDQS7+: U5.F3 (LDQS)
- new net DRAM_SDQS7-: U5.G3 (~LDQS)
