File: Design_IMX6QP/IMXDesign/Power.sch (KiCad schematic (older format))
At the start: 69 parts, among them U7 W_MMPF0100

Commit message: Update IMX6QP and IMX8MQ
Parts:
- L1, L6: value 1uH -> 1u/3.9A; footprint Inductor_SMD:L_2816_7142Metric -> Inductor_SMD:L_Vishay_IHLP-1212
- L2, L4, L5: value 1uH -> 1u/2.6A; footprint Inductor_SMD:L_2816_7142Metric -> Inductor_SMD:L_TDK_NLV25_2.5x2.0mm
- U7: symbol William_IMX6QP:W_MMPF0100 -> IMXDesign-rescue:W_MMPF0100-William_IMX6QP
Connections:
- net +1v375_SOC renamed +1V375_CORE
- net +1V375_CORE: no longer C59.1, C60.1, C61.1, L6.2, TP3.1, U7.6 (SW1FB)
- new net +1V375_SOC: C59.1, C60.1, C61.1, L6.2, TP3.1, U7.6 (SW1FB)
Other:
- moved on the sheet: C15, C16, C17, C18, C19, C22, C23, C24, C25, C26, C27, C28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
