File: Design_IMX6QP/IMXDesign/eMMC.sch (KiCad schematic (older format))
At the start: 9 parts, among them U6 MTFC16GAKAECN-4M_IT

Commit message: Update IMX6QP and IMX8MQ
Parts:
- U6: symbol MTFC16GAKAECN-4M_IT:MTFC16GAKAECN-4M_IT -> IMXDesign-rescue:MTFC16GAKAECN-4M_IT-MTFC16GAKAECN-4M_IT
Connections:
- net SD_CMD: now reaches U6.M5 (CMD)
Other:
- moved on the sheet: C64, C65, C66, C67, C68, C69, C70, C71, U6A, U6B
