File: Design_IMX8Q/Base_Board/IMX8MQ/Power_IMX8.kicad_sch (KiCad schematic)
At the start: 1 part, among them U1 MIMX8MQ6CVAHZAB

Commit message: Add QSPI and more color
Parts:
- removed U1: MIMX8MQ6CVAHZAB, IMX8MQ_footprints:MIMX8MQ6CVAHZAB, symbol _MIMX8MQ6CVAHZAB:MIMX8MQ6CVAHZAB
- added C1, C10, C2, C3, C4, C5, C6, C7, C8, C9: 4.7uF, Capacitor_SMD:C_0402_1005Metric, symbol Device:C_Small
- added C11, C12, C13: 22uF, Capacitor_SMD:C_0805_2012Metric, symbol Device:C_Small
- added C14: 22uF, Capacitor_SMD:C_0402_1005Metric, symbol Device:C_Small
- added C15, C16: 10uF, Capacitor_SMD:C_0805_2012Metric, symbol Device:C_Small
- added C17, C64, C65, C66: 0.1uF, Capacitor_SMD:C_0402_1005Metric, symbol Device:C_Small
- added C18, C63: 1uF, Capacitor_SMD:C_0402_1005Metric, symbol Device:C_Small
- added C31, C32, C33, C34, C35, C36, C37, C38, C39, C40, C41, C42, C43, C44, C45, C46, C47, C55, C56, C57, C58: 22uF, Capacitor_SMD:C_0603_1608Metric, symbol Device:C_Small
- added C48, C49, C50, C51, C52, C53: 4.7uF, Capacitor_SMD:C_0603_1608Metric, symbol Device:C_Small
- added C54: 1uF, Capacitor_SMD:C_0603_1608Metric, symbol Device:C_Small
- added C59: 220uF, symbol Device:C_Polarized_Small
- added C60, C61, C62: 0.47uF, Capacitor_SMD:C_0402_1005Metric, symbol Device:C_Small
- added L1: 1.5uH, Inductor_SMD:L_7.3x7.3_H4.5, symbol Device:L_Small
- added L2: 4.7uH, Inductor_SMD:L_Taiyo-Yuden_NR-40xx, symbol Device:L_Small
- added L3, L4, L5, L6, L7: 1uH, Inductor_SMD:L_Taiyo-Yuden_NR-30xx_HandSoldering, symbol Device:L_Small
- added Q1: AO3401A, Package_TO_SOT_SMD:SOT-23, symbol Transistor_FET:AO3401A
- added R3: 1.5M, Resistor_SMD:R_0402_1005Metric, symbol Device:R_Small
- added R4: 44.2K, Resistor_SMD:R_0402_1005Metric, symbol Device:R_Small
- added R5: 9.53k, Resistor_SMD:R_0402_1005Metric, symbol Device:R_Small
- added R6, R7: 100k, Resistor_SMD:R_0402_1005Metric, symbol Device:R_Small
- added R8: 10K, Resistor_SMD:R_0402_1005Metric, symbol Device:R_Small
- added U3: ~, Package_DFN_QFN:QFN-56-1EP_8x8mm_P0.5mm_EP4.3x4.3mm, symbol _W_MX8M:MC34PF4210
- added U4: MP8759GD-Z, _W_SBC:MP8759GD-Z, symbol MP8759GD-Z:MP8759GD-Z
- added U5: MP2263GD-Z, _W_SBC:MP2263, symbol MP2263:MP2263GD-Z
Connections:
- net GND: now also C1.2, C10.2, C11.2, C12.2, C13.2, C14.2, C15.2, C16.2, C17.2, C18.2, C2.2, C3.2, C31.2, C32.2, C33.2, C34.2, C35.2, C36.2, C37.2, C38.2, C39.2, C4.2, C40.2, C41.2, C42.2, C43.2, C44.2, C45.2, C46.2, C47.2, C48.2, C49.2, C5.2, C50.2, C51.2, C52.2, C53.2, C54.2, C55.2, C56.2, C57.2, C58.2, C59.2, C6.2, C60.2, C61.2, C62.2, C63.2, C64.2, C66.2, C7.2, C8.2, C9.2, R5.2, R7.2, U3.15 (GNDREF1), U3.32 (SW3VSSSNS), U3.48 (GNDREF), U3.57 (EPGND), U4.10 (AGND), U4.2 (PGND), U5.12 (AGND), U5.3 (PGND), U5.8 (PGND)
- new net: C18.1, R8.1, U5.11 (VCC)
- new net: C52.1, U3.41 (VGEN6)
- new net: C42.1, C43.1, C44.1, C45.1, L6.2, U3.38 (SW3AFB)
- new net: C51.1, U3.28 (VGEN4)
- new net: C65.2, C66.1, U3.29 (VHALF)
- new net: C50.1, U3.26 (VGEN3)
- new net: R8.2, U5.6 (PG)
- new net: L7.1, U3.21 (SW4LX)
- new net: C54.1, U3.31 (VREFDDR)
- new net: R4.2, R5.1, U4.11 (FB)
- new net: R3.1, U4.12 (EN)
- new net: R6.2, R7.1, U4.6 (MODE)
- new net: L1.1, U4.7 (SW)
- new net: C14.1, R6.1, U4.9 (VCC)
- new net: L4.1, U3.11 (SW1CLX), U3.14 (SW1VSSSNS)
- new net: C48.1, U3.16 (VGEN1)
- new net: C49.1, U3.18 (VGEN2)
- new net: C62.1, U3.40 (VIN3)
- new net: C64.1, U3.42 (LICELL)
- new net: C53.1, U3.43 (VSNVS)
- new net: L6.1, U3.35 (SW3BLX), U3.36 (SW3ALX)
- new net: L2.1, U5.9 (SW)
- new net: L3.1, U3.8 (SW1ALX), U3.9 (SW1BLX)
- new net: L5.1, U3.22 (SW2LX)
- new net DCDC_3V3: C1.1, C10.1, C2.1, C3.1, C4.1, C5.1, C55.1, C56.1, C57.1, C58.1, C59.1, C6.1, C60.1, C61.1, C63.1, C7.1, C8.1, C9.1, L1.2, Q1.3 (D), R4.1, U3.10 (SW1BIN), U3.12 (SW1CIN), U3.17 (VIN1), U3.20 (SW4IN), U3.23 (SW2IN), U3.24 (SW2IN), U3.27 (VIN2), U3.34 (SW3BIN), U3.37 (SW3AIN), U3.45 (SWBSTIN), U3.50 (VIN), U3.7 (SW1AIN), U4.5 (VOUT)
- new net DCDC_5V: L2.2
- new net NVCC_DRAM_1V1: C38.1, C39.1, C40.1, C65.1, L5.2, U3.25 (SW2FB), U3.30 (VINREFDDR)
- new net NVCC_SD1_1V8: C41.1, C46.1, C47.1, L7.2, U3.19 (SW4FB)
- new net VDD_3V3: Q1.2 (S)
- new net VDD_GPU_0V9: C31.1, C32.1, C33.1, C34.1, L3.2, U3.6 (SW1FB)
- new net VDD_VPU_0V9: C35.1, C36.1, C37.1, L4.2, U3.13 (SW1CBF)
- new net VSYS: C11.1, C12.1, C13.1, C15.1, C16.1, C17.1, R3.2, U4.1 (VIN), U5.2 (VIN)
Other:
- note added: "10v"
- note added: "25v"
- note added: "35v"
- note added: "50v"

Commit message: it was inserted power control system
Parts:
- removed C40: 22uF, Capacitor_SMD:C_0603_1608Metric, symbol Device:C_Small
- added C11 (x2), C12 (x2), C13 (x2): 22uF, Capacitor_SMD:C_0805_2012Metric, symbol Device:C_Small
- added C15 (x3), C16 (x3): 10uF, Capacitor_SMD:C_0805_2012Metric, symbol Device:C_Small
- added C17 (x3): 5.6uF, Capacitor_SMD:C_0402_1005Metric, symbol Device:C_Small
- added C17 (x3): 0.1uF, Capacitor_SMD:C_0402_1005Metric, symbol Device:C_Small
- added C18 (x3): 1uF, Capacitor_SMD:C_0402_1005Metric, symbol Device:C_Small
- added C39: 22uF, Capacitor_SMD:C_0603_1608Metric, symbol Device:C_Small
- added C48, C50: 1uF, Capacitor_SMD:C_0603_1608Metric, symbol Device:C_Small
- added C49: 0.22uF, Capacitor_SMD:C_0603_1608Metric, symbol Device:C_Small
- added L2 (x2): 4.7uH, Inductor_SMD:L_Taiyo-Yuden_NR-40xx, symbol Device:L_Small
- added R3: 10.0k, Resistor_SMD:R_0402_1005Metric, symbol Device:R_Small
- added R8 (x6): 10K, Resistor_SMD:R_0402_1005Metric, symbol Device:R_Small
- added R8 (x3): 0K, Resistor_SMD:R_0402_1005Metric, symbol Device:R_Small
- added R8: 27K, Resistor_SMD:R_0402_1005Metric, symbol Device:R_Small
- added U16, U17: MP2147GD-P, _W_SBC:MP2147GD-P, symbol MP2147GD-P:MP2147GD-P
- added U18: UM805RE, _W_SBC:UM805RE, symbol UM805RE:UM805RE
- added U19: LDCL015MR, _W_SBC:LDCL015MR, symbol LDCL015MR:LDCL015MR
- L1: footprint Inductor_SMD:L_7.3x7.3_H4.5 -> Inductor_SMD:L_Taiyo-Yuden_NR-60xx_HandSoldering
Connections:
- net DCDC_3V3: now also C11.1, C11.1, C12.1, C12.1, C13.1, C13.1, U16.13 (VIN), U16.8 (VIN), U17.13 (VIN), U17.8 (VIN)
- net DCDC_5V: now also C15.1, C16.1, C17.1, R8.2
- net GND: now also C11.2, C11.2, C12.2, C12.2, C13.2, C13.2, C15.2, C15.2, C15.2, C16.2, C16.2, C16.2, C17.2, C17.2, C17.2, C18.2, C18.2, C39.2, C48.1, C49.1, C50.1, R3.1, R8.1, R8.1, R8.1, R8.1, U16.10 (GND), U16.11 (GND), U16.12 (GND), U17.10 (GND), U17.11 (GND), U17.12 (GND)
- net NVCC_DRAM_1V1: now also C39.1
- net VDD_3V3: now also R8.1
- net VCAM_2V8: now reaches C52.1, U3.41 (VGEN6)
- net VDD_DRAM_0V9: now reaches C42.1, C43.1, C44.1, C45.1, L6.2, U3.38 (SW3AFB)
- net VDDA_1V8: now reaches C51.1, U3.28 (VGEN4)
- net VDD_PHY_1V8: now reaches C50.1, U3.26 (VGEN3)
- net VREFDDR: now reaches C54.1, U3.31 (VREFDDR)
- net POR_B: now reaches U3.3 (/RESETBMCU)
- net at U3.47 (VDDOTP): now also R3.2
- net at U3.49 (VCORE): now also C50.2
- net at U3.51 (VCOREDIG): now also C48.2
- net at U3.52 (VCOREREF): now also C49.2
- net NVCC_3V3: now reaches U3.55 (VDDIO)
- net VCAM_1V5: now reaches C48.1, U3.16 (VGEN1)
- net VDD_PHY_0V9: now reaches C49.1, U3.18 (VGEN2)
- net VDD_PHY_3V3: now reaches U3.39 (VGEN5)
- net VDD_SNVS_0V9: now reaches C53.1, U3.43 (VSNVS)
- net VDD_SNVS_0V9: now also U19.5 (VOUT)
- net at U5.10 (BST): now also C18.1
- net at U5.13 (SS): now also C18.1
- net at U5.14 (FB): now also R8.1
- net at U5.15 (FREQ): now also R8.2
- net at U5.4 (EN): now also R8.2
- net at U5.7 (BIAS): now also C18.1
- net at L2.1, U5.9 (SW): now also C18.2
- new net: C17.2, R8.1, R8.2
- new net: C17.1, R8.1, R8.2, R8.2
- new net: C17.2, U16.4 (RAMP)
- new net: L2.1, U16.1 (SW), U16.9 (SW)
- new net: C17.2, U17.4 (RAMP)
- new net: U17.5 (EN), U18.2 (RESET)
- new net: R8.1, R8.2, U16.7 (PG)
- new net: L2.1, U17.1 (SW), U17.9 (SW)
- new net: R8.1, R8.2, U17.7 (PG)
- new net VDD_ARM_0V9: C15.1, C16.1, C17.1, C17.1, L2.2, R8.2, U16.2 (OUT)
- new net VDD_SOC_0V9: C15.1, C16.1, C17.1, C17.1, L2.2, R8.2, U17.2 (OUT)
Other:
- moved on the sheet: C1, C10, C11, C12, C13, C14, C15, C16, C17, C18, C2, C3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
