File: LoRa/LR1121/LR1121/LoRa-system.kicad_sch (KiCad schematic)
At the start: 44 parts, among them J1 USB_B_Micro, J2 Con_GPS, SW1 NRST, SW2 BOOT0, U1 LBAA0XV2GT, U2 STM32L552CCUx, U3 MT29F4G01ABAFDWB-IT:F TR, U4 PCMF1USB3S, U5 MAX-M10S, U6 LTC4162IUFD-FFSM_PBF, Y1 32.768KHz, Y2 25MHz

Commit message: [PCB] Inster power module in the PCB
It was improve the power module
.
Parts:
- added C19, C21: 100nF, Capacitor_SMD:C_0402_1005Metric, symbol Device:C_Small
- added C22, C23: 10uF, Capacitor_SMD:C_1206_3216Metric, symbol Device:C_Small
- added C24: 150uF, Capacitor_Tantalum_SMD:CP_EIA-1608-10_AVX-L, symbol Device:C_Polarized_Small
- added C25: 0.022uF, Capacitor_SMD:C_0402_1005Metric, symbol Device:C_Small
- added D3: RED, LED_SMD:LED_0402_1005Metric, symbol Device:LED_Small
- added L2: 6.8uH, Inductor_SMD:L_Coilcraft_XAL6060-XXX, symbol Device:L_Small
- added Q1, Q2: FDMC8327L, _W_LoRa:WDFN8_511DR_OSI, symbol FDMC8327L:FDMC8327L
- added R10, R11, R12, R13, R14, R15: 0, Resistor_SMD:R_0603_1608Metric, symbol Device:R_Small
- added R16: 2.2K, Resistor_SMD:R_0402_1005Metric, symbol Device:R_Small
- added R17, R18: 4.7K, Resistor_SMD:R_0402_1005Metric, symbol Device:R_Small
- added R19: 100K, Resistor_SMD:R_0402_1005Metric, symbol Device:R_Small
- added R20: 63.4K, Resistor_SMD:R_0603_1608Metric, symbol Device:R_Small
- added R21: 10K, Resistor_SMD:R_0603_1608Metric, symbol Device:R_Small
- added R22, R23: 10k, Resistor_SMD:R_0603_1608Metric, symbol Device:R_Small
- added R8, R9: 0.01, Resistor_SMD:R_0603_1608Metric, symbol Device:R_Small
Connections:
- net GND: now also U6.23 (PGND), U6.24 (PGND), U6.29 (AGND), C19.2, C21.2, C22.2, C23.2, C24.2, R10.1, R15.1, R20.2, R21.2, R23.2
- net BOOST: now reaches U6.1 (BOOST)
- net BOOST: now also C25.1
- net NTC: now reaches U6.10 (NTC)
- net NTC: now also R22.2, R23.1
- net at U6.11 (RT): now also R20.1
- net SMBALERT#: now reaches U6.12 (~{SMBALERT})
- net SMBALERT#: now also D3.1 (K), R19.2
- net I2C_SCL_MIC: now reaches U6.13 (SCL)
- net I2C_SCL_MIC: now also R17.2
- net I2C_SDA_MIC: now reaches U6.14 (SDA)
- net I2C_SDA_MIC: now also R18.2
- net DVCC: now reaches U6.15 (DVCC)
- net DVCC: now also R16.1, R17.1, R18.1, R19.1
- net SYNC: now reaches U6.16 (SYNC)
- net SYNC: now also R21.1
- net CELLS0: now reaches U6.17 (CELLS0)
- net CELLS0: now also R10.2, R11.2, R12.2
- net CELLS1: now reaches U6.18 (CELLS1)
- net CELLS1: now also R13.2, R14.2, R15.2
- net BATSENS+: now reaches U6.19 (BATSENS+)
- net BATSENS+: now also U6.20 (CSN), C23.1, C24.1, R9.2
- net INTVCC: now reaches U6.2 (INTVCC)
- net INTVCC: now also R12.1, R13.1
- net CSP: now reaches U6.21 (CSP)
- net CSP: now also L2.1, Q2.5, Q2.6, Q2.7, Q2.8, R9.1
- net BATFET: now reaches U6.22 (BATFET)
- net BATFET: now also Q2.4
- net SW: now reaches U6.25 (SW), U6.26 (SW)
- net SW: now also C25.2, L2.2
- net CLN: now reaches U6.27 (VOUT), U6.28 (VOUT)
- net CLN: now also U6.3 (VOUTA), U6.4 (CLN), C21.1, C22.1, Q2.1, Q2.2, Q2.3, R8.2
- net CLP: now reaches U6.5 (CLP)
- net CLP: now also Q1.5, Q1.6, Q1.7, Q1.8, R8.1
- net at U6.6 (INFET): now also Q1.4
- net VIN: now reaches U6.7 (VIN)
- net VIN: now also C19.1, Q1.1, Q1.2, Q1.3
- net VCC2P5: now reaches U6.8 (VCC2P5)
- net VCC2P5: now also R11.1, R14.1
- net NTCBIAS: now reaches U6.9 (NTCBIAS)
- net NTCBIAS: now also R22.1
- new net: D3.2 (A), R16.2
Other:
- moved on the sheet: U6

Commit message: [PMIC] Changes PMIC chip to LTC4146 for BQ25619
The BQ25619 is now the PMIC because it had 3.5v-4.5v
Parts:
- removed C24: 150uF, Capacitor_Tantalum_SMD:CP_EIA-1608-10_AVX-L, symbol Device:C_Polarized_Small
- removed D3: RED, LED_SMD:LED_0402_1005Metric, symbol Device:LED_Small
- removed Q1, Q2: FDMC8327L, _W_LoRa:WDFN8_511DR_OSI, symbol FDMC8327L:FDMC8327L
- removed R15: 0, Resistor_SMD:R_0603_1608Metric, symbol Device:R_Small
- removed R16: 2.2K, Resistor_SMD:R_0402_1005Metric, symbol Device:R_Small
- removed R17, R18: 4.7K, Resistor_SMD:R_0402_1005Metric, symbol Device:R_Small
- removed R19: 100K, Resistor_SMD:R_0402_1005Metric, symbol Device:R_Small
- removed R20: 63.4K, Resistor_SMD:R_0603_1608Metric, symbol Device:R_Small
- removed R21: 10K, Resistor_SMD:R_0603_1608Metric, symbol Device:R_Small
- removed R22, R23: 10k, Resistor_SMD:R_0603_1608Metric, symbol Device:R_Small
- removed U6: LTC4162IUFD-FFSM_PBF, _W_LoRa:QFN50P500X400X80-29N, symbol LTC4162IUFD-FFSM_PBF:LTC4162IUFD-FFSM_PBF
- added C24: 0.047uF, Capacitor_SMD:C_0402_1005Metric, symbol Device:C_Small
- added U7: BQ25619ERTWR, _W_LoRa:BQ25619ERTWR, symbol BQ25619ERTWR:BQ25619ERTWR
- C19: value 100nF -> 1uF
- C21: value 100nF -> 10uF; footprint Capacitor_SMD:C_0402_1005Metric -> Capacitor_SMD:C_0805_2012Metric
- C22, C23: footprint Capacitor_SMD:C_1206_3216Metric -> Capacitor_SMD:C_0805_2012Metric
- C25: value 0.022uF -> 0.1uF
- L2: value 6.8uH -> 2.2uH; footprint Inductor_SMD:L_Coilcraft_XAL6060-XXX -> Inductor_SMD:L_Taiyo-Yuden_MD-4040
- R10, R12: value 0 -> 10K; footprint Resistor_SMD:R_0603_1608Metric -> Resistor_SMD:R_0402_1005Metric
- R11, R13, R14: value 0 -> 0.01; footprint Resistor_SMD:R_0603_1608Metric -> Resistor_SMD:R_2010_5025Metric
- R8, R9: value 0.01 -> 10K; footprint Resistor_SMD:R_0603_1608Metric -> Resistor_SMD:R_0402_1005Metric
Connections:
- net GND: now also C25.2, R12.2, U7.17 (PGND), U7.18 (PGND), U7.25 (PAD); no longer R10.1
- net VIN: now also J1.1 (VBUS); no longer C19.1
- net BATSENS+: no longer names the net of C23.1
- net BATSENS+: now also R13.1, U7.13 (BAT), U7.14 (BAT); no longer R9.2
- net BOOST: no longer names the net of C25.1
- net BOOST: now also U7.10 (BATSNS)
- removed net CELLS0: R10.2, R11.2, R12.2
- net CELLS1: no longer names the net of R14.2
- net CELLS1: no longer R13.2
- net CLN: no longer names the net of C21.1, C22.1
- net CLN: now also L2.1, R14.1, U7.15 (SYS), U7.16 (SYS); no longer R8.2
- net CLP: no longer names the net of R8.1
- net CLP: now also R10.1, R9.1
- removed net CSP: L2.1, R9.1
- net INTVCC: no longer names the net of R12.1
- net INTVCC: now also C19.1, R11.2, U7.1 (VAC), U7.24 (VBUS); no longer R13.1
- net SW: no longer names the net of L2.2
- net SW: now also C24.1, U7.19 (SW), U7.20 (SW); no longer C25.2
- net VCC2P5: no longer names the net of R11.1
- net VCC2P5: no longer R14.1
- new net: R9.2, U7.6 (SDA)
- new net: C24.2, U7.21 (BTST)
- new net: R8.2, U7.9 (CE_N)
- new net: R10.2, U7.5 (SCL)
- new net INT_N: U7.7 (INT_N)
- new net REGN: U7.22 (REGN)
- new net TS: U7.11 (TS)
- no-connect marks 4 -> 5

Commit message: [BB_IMX8ML] Change MCU F280015x
Change MCU STM32H5 for F2800157 dual core real-time
Parts:
- removed AE1: 2.4Gz, Connector_Coaxial:SMA_Molex_73251-1153_EdgeMount_Horizontal, symbol Device:Antenna
- removed AE2: SUB-GHz, Connector_Coaxial:SMA_Molex_73251-1153_EdgeMount_Horizontal, symbol Device:Antenna
- removed AE3: GPS, Connector_Coaxial:U.FL_Hirose_U.FL-R-SMT-1_Vertical, symbol Device:Antenna
- removed C1, C2, C3, C4: NU, Capacitor_SMD:C_0402_1005Metric, symbol Device:C_Small
- removed C10, C11, C12, C14, C15, C16, C17, C18, C20: 100nF, Capacitor_SMD:C_0402_1005Metric, symbol Device:C_Small
- removed C13: 2.2uF, Capacitor_Tantalum_SMD:CP_EIA-1608-08_AVX-J, symbol Device:C_Polarized_Small
- removed C19: 1uF, Capacitor_SMD:C_0402_1005Metric, symbol Device:C_Small
- removed C21, C22, C23: 10uF, Capacitor_SMD:C_0805_2012Metric, symbol Device:C_Small
- removed C24: 0.047uF, Capacitor_SMD:C_0402_1005Metric, symbol Device:C_Small
- removed C25: 0.1uF, Capacitor_SMD:C_0402_1005Metric, symbol Device:C_Small
- removed C5, C6, C7, C8: 12pF, Capacitor_SMD:C_0402_1005Metric, symbol Device:C_Small
- removed C9: 10uF, Capacitor_SMD:C_0603_1608Metric, symbol Device:C_Small
- removed D1: GREEN, LED_SMD:LED_0402_1005Metric, symbol Device:LED_Small
- removed D2: RED, LED_SMD:LED_0402_1005Metric, symbol Device:LED_Small
- removed J1: USB_B_Micro, Connector_USB:USB_Mini-B_Wuerth_65100516121_Horizontal, symbol Connector:USB_B_Micro
- removed J2: Con_GPS, Connector_PinSocket_2.54mm:PinSocket_2x02_P2.54mm_Vertical, symbol Connector_Generic:Conn_02x02_Odd_Even
- removed L1: 27nH, Inductor_SMD:L_0402_1005Metric, symbol Device:L_Small
- removed L2: 2.2uH, Inductor_SMD:L_Taiyo-Yuden_MD-4040, symbol Device:L_Small
- removed R1, R2: 0, Resistor_SMD:R_0402_1005Metric, symbol Device:R_Small
- removed R10, R12, R3, R8, R9: 10K, Resistor_SMD:R_0402_1005Metric, symbol Device:R_Small
- removed R11, R13, R14: 0.01, Resistor_SMD:R_2010_5025Metric, symbol Device:R_Small
- removed R4, R5, R6, R7: 100, Resistor_SMD:R_0402_1005Metric, symbol Device:R_Small
- removed SW1: NRST, Button_Switch_SMD:SW_Push_1P1T_XKB_TS-1187A, symbol Switch:SW_SPST
- removed SW2: BOOT0, Button_Switch_SMD:SW_Push_1P1T_XKB_TS-1187A, symbol Switch:SW_SPST
- removed U1: LBAA0XV2GT, _W_LoRa:LBAA0XV2GT, symbol _W_LoRa:LBAA0XV2GT-001
- removed U2: STM32L552CCUx, Package_DFN_QFN:QFN-48-1EP_7x7mm_P0.5mm_EP5.6x5.6mm, symbol MCU_ST_STM32L5:STM32L552CCUx
- removed U3: MT29F4G01ABAFDWB-IT:F TR, _W_LoRa:SON127P600X800X65-8N, symbol Memory_EEPROM:CAT250xxx
- removed U4: PCMF1USB3S, _W_SBC:WLCSP52-1-2_NEX, symbol _W_MX8M:PCMF1HDMI2S
- removed U5: MAX-M10S, RF_GPS:ublox_MAX, symbol RF_GPS:MAX-M10S
- removed U7: BQ25619ERTWR, _W_LoRa:BQ25619ERTWR, symbol BQ25619ERTWR:BQ25619ERTWR
- removed Y1: 32.768KHz, Crystal:Crystal_SMD_3215-2Pin_3.2x1.5mm, symbol Device:Crystal_Small
- removed Y2: 25MHz, Crystal:Crystal_SMD_3225-4Pin_3.2x2.5mm, symbol Device:Crystal_GND24_Small
Connections:
- no-connect marks 5 -> 0
Other:
- added sheet ComunicationUnit (comunication_unit.kicad_sch)
- added sheet ControlUnit (control_unit.kicad_sch)
- added sheet PowerUnit (power_unit.kicad_sch)
