File: Design_IMX8ML_Plus/BB_IMX8MLP/BB_IMX8MLP/connector_left.kicad_sch (KiCad schematic)
At the start: 8 parts, among them J26 DF40C-80DP-0.4V_51_, J31 Front_Right

Commit message: [IMX8ML] Add new layer
A new layers was add in the cpu schematic, now it had 8 layer.
Connections:
- net EARC_AUX: now also J26.3; no longer J26.4
- net EARC_N_HPD: now also J26.5; no longer J26.6
- net EARC_P_UTIL: now also J26.7; no longer J26.8
- net ECSPI1_MISO: now also J31.70; no longer J31.69
- net ECSPI1_MOSI: now also J31.72; no longer J31.71
- net ECSPI1_SCLK: now also J31.74; no longer J31.73
- net ECSPI1_SSO: now also J31.76; no longer J31.75
- net ECSPI2_MISO: now also J31.78; no longer J31.77
- net ECSPI2_MOSI: now also J31.80; no longer J31.79
- net ECSPI2_SCLK: now also J31.82; no longer J31.81
- net ECSPI2_SSO: now also J31.84; no longer J31.83
- net ENET_MDC: now also J26.55; no longer J26.44
- net ENET_MDIO: now also J26.57; no longer J26.46
- net ENET_RD0: now also J26.45; no longer J26.34
- net ENET_RD1: now also J26.43; no longer J26.40
- net ENET_RD2: now also J26.41; no longer J26.42
- net ENET_RD3: now also J26.39; no longer J26.26
- net ENET_TD0: now also J26.27; no longer J26.32
- net ENET_TD1: now also J26.29; no longer J26.38
- net ENET_TD2: now also J26.31; no longer J26.36
- net ENET_TD3: now also J26.33; no longer J26.28
- net ETH1_LED1: now also J31.67; no longer J31.8
- net ETH1_LED2: now also J31.69; no longer J31.10
- net ETH1_MDI0+: now also J31.93; no longer J31.34
- net ETH1_MDI0-: now also J31.91; no longer J31.32
- net ETH1_MDI1+: now also J31.87; no longer J31.28
- net ETH1_MDI1-: now also J31.85; no longer J31.26
- net ETH1_MDI2+: now also J31.81; no longer J31.22
- net ETH1_MDI2-: now also J31.79; no longer J31.20
- net ETH1_MDI3+: now also J31.75; no longer J31.16
- net ETH1_MDI3-: now also J31.73; no longer J31.14
- net HDMI_CEC: now also J31.22; no longer J31.25
- net HDMI_DDC_SCL: now also J31.8; no longer J31.33
- net HDMI_DDC_SDA: now also J31.10; no longer J31.31
- net HDMI_HPD: now also J31.20; no longer J31.27
- net HDMI_TX0_N: now also J31.26; no longer J31.21
- net HDMI_TX0_P: now also J31.28; no longer J31.19
- net HDMI_TX1_N: now also J31.32; no longer J31.15
- net HDMI_TX1_P: now also J31.34; no longer J31.13
- net HDMI_TX2_N: now also J31.38; no longer J31.9
- net HDMI_TX2_P: now also J31.40; no longer J31.7
- net HDMI_TXC_N: now also J31.14; no longer J31.39
- net HDMI_TXC_P: now also J31.16; no longer J31.37
- net I2C1_SCL: now also J26.18; no longer J26.17
- net I2C1_SDA: now also J26.20; no longer J26.19
- net I2C2_SCL: now also J26.30; no longer J26.29
- net I2C2_SDA: now also J26.32; no longer J26.31
- net I2C3_SCL: now also J26.26; no longer J26.25
- net I2C3_SDA: now also J26.24; no longer J26.23
- net I2C4_SCL: now also J26.38; no longer J26.37
- net I2C4_SDA: now also J26.36; no longer J26.35
- net SAI1_MCLK: now also J26.2; no longer J26.1
- net SAI1_RXC: now also J26.4; no longer J26.3
- net SAI1_RXD0: now also J26.13; no longer J26.14
- net SAI1_RXD1: now also J26.11; no longer J26.12
- net SAI1_RXFS: now also J26.6; no longer J26.5
- net SAI1_TXC: now also J26.49; no longer J26.22
- net SAI1_TXD4: now also J26.37; no longer J26.20
- net SAI1_TXD5: now also J26.35; no longer J26.16
- net SAI1_TXD6: now also J26.23; no longer J26.24
- net SAI1_TXD7: now also J26.17; no longer J26.18
- net SAI1_TXFS: now also J26.10; no longer J26.9
- net SAI2_MCLK: now also J31.21; no longer J31.64
- net SAI2_RXC: now also J31.23; no longer J31.66
- net SAI2_RXD0: now also J31.33; no longer J31.76
- net SAI2_RXFS: now also J31.25; no longer J31.68
- net SAI2_TXC: now also J31.27; no longer J31.70
- net SAI2_TXD0: now also J31.35; no longer J31.78
- net SAI2_TXFS: now also J31.29; no longer J31.72
- net SAI3_MCLK: now also J31.5; no longer J31.48
- net SAI3_RXC: now also J31.7; no longer J31.50
- net SAI3_RXD: now also J31.9; no longer J31.52
- net SAI3_RXFS: now also J31.11; no longer J31.54
- net SAI3_TXC: now also J31.13; no longer J31.56
- net SAI3_TXD: now also J31.15; no longer J31.58
- net SAI3_TXFS: now also J31.17; no longer J31.60
- net SAI5_MCLK: now also J31.51; no longer J31.94
- net SAI5_RXC: now also J31.41; no longer J31.84
- net SAI5_RXD0: now also J31.43; no longer J31.86
- net SAI5_RXD1: now also J31.45; no longer J31.88
- net SAI5_RXD2: now also J31.47; no longer J31.90
- net SAI5_RXD3: now also J31.49; no longer J31.92
- net SAI5_RXFS: now also J31.53; no longer J31.96
- net SDC1_RESET_B: now also J31.55
- net SDC2_CD_B: now also J31.54; no longer J31.53
- net SDC2_CLK: now also J31.46; no longer J31.45
- net SDC2_CMD: now also J31.48; no longer J31.47
- net SDC2_DATA0: now also J31.52; no longer J31.51
- net SDC2_DATA1: now also J31.50; no longer J31.49
- net SDC2_DATA2: now also J31.56; no longer J31.55
- net SDC2_DATA3: now also J31.58; no longer J31.57
- net SDC2_RESET_B: now also J31.60; no longer J31.59
- net SDC2_WP: now also J31.62; no longer J31.61
- net UART1_RXD: now also J26.46; no longer J26.45
- net UART1_TXD: now also J26.44; no longer J26.43
- net UART2_RXD: now also J26.40; no longer J26.39
- net UART2_TXD: now also J26.42; no longer J26.41
- net UART4_RXD: now also J26.48; no longer J26.47
- net UART4_TXD: now also J26.50; no longer J26.49
- net ON/OFF: no longer names the net of J26.51
- net PMIC_RST_B: no longer names the net of J26.53
Other:
- note added: "ETH_2_RGMII_RXC_CTL"
