File: Design_IMX8ML_Plus/BB_IMX8MLP/BB_IMX8MLP/serial_interface.kicad_sch (KiCad schematic)
At the start: 1 part, among them U31 FT4232H

Commit message: Review
Parts:
- added C139, C141, C158, C160, C161, C162, C163, C164, C165, C166, C167: 100nF, Capacitor_SMD:C_0402_1005Metric, symbol Device:C_Small
- added C140, C157, C159, C170: 10uF, Capacitor_SMD:C_0402_1005Metric, symbol Device:C_Small
- added C168, C169: 1nF, Capacitor_SMD:C_0402_1005Metric, symbol Device:C_Small
- added J23: USB_C_Receptacle, symbol Connector:USB_C_Receptacle
- added R46, R68, R70: 10k, Resistor_SMD:R_0402_1005Metric, symbol Device:R_Small
- added R69: 12k, Resistor_SMD:R_0402_1005Metric, symbol Device:R_Small
- added U22: PCMF3USB3S, Package_CSP:Nexperia_WLCSP-15_6-3-6_2.37x1.17mm_Layout6x3_P0.4mm, symbol Power_Protection:PCMF3USB3S
- added U32, U34: ~, symbol _W_MX8M:SN74AVC4T774RSVR
- added U33: TJA1052i-1, Package_SO:SOIC-16W_7.5x10.3mm_P1.27mm, symbol Interface_CAN_LIN:TJA1052i-1
- U31: footprint (none) -> Package_DFN_QFN:VQFN-64-1EP_9x9mm_P0.5mm_EP5.4x5.4mm
Connections:
- net GND: now reaches U31.1 (GND)
- net GND: now also U31.10 (AGND), U31.11 (GND), U31.15 (GND), U31.25 (GND), U31.35 (GND), U31.47 (GND), U31.5 (GND), U31.51 (GND), C139.2, C141.2, C158.2, C159.2, C160.2, C161.2, C162.2, C163.2, C164.2, C165.2, C166.2, C167.2, C168.2, C169.2, R46.2, R68.2, R69.2, R70.2, U22.B2 (GND_CH2), U32.8 (GND), U32.9 (GND), U34.8 (GND), U34.9 (GND)
- net at U31.12 (VCORE): now also U31.37 (VCORE), U31.64 (VCORE)
- net at U31.14 (~{RESET}): now also R69.1
- net at U31.20 (VCCIO): now also U31.31 (VCCIO), U31.42 (VCCIO), U31.56 (VCCIO)
- net mcu_UARTA_3V3_TXD: now reaches U31.21 (ADBUS4)
- net mcu_UARTA_3V3_RXD: now reaches U31.22 (ADBUS5)
- net mcu_UARTA_3V3_RTC: now reaches U31.23 (ADBUS6)
- net mcu_UARTA_3V3_CTS: now reaches U31.24 (ADBUS7)
- net FTDI_JTAG_TCK: now reaches U31.26 (BDBUS0)
- net FTDI_JTAG_TCK: now also U32.12 (1B1)
- net FTDI_JTAG_TDI: now reaches U31.27 (BDBUS1)
- net FTDI_JTAG_TDI: now also U32.11 (1B2)
- net FTDI_JTAG_TDO: now reaches U31.28 (BDBUS2)
- net FTDI_JTAG_TDO: now also U32.10 (2B1)
- net FTDI_JTAG_TMS: now reaches U31.29 (BDBUS3)
- net FTDI_JTAG_TMS: now also U32.9 (GND)
- net FTDI_JTAG_TRST#: now reaches U31.30 (BDBUS4)
- net FTDI_UARTC_3V3_TXD: now reaches U31.38 (CDBUS0)
- net FTDI_UARTC_3V3_TXD: now also U34.12 (1B1)
- net FTDI_UARTC_3V3_RXD: now reaches U31.39 (CDBUS1)
- net FTDI_UARTC_3V3_RXD: now also U34.11 (1B2)
- net at U31.4 (VPHY): now also U31.9 (VPLL)
- net FTDI_UARTC_3V3_RTC: now reaches U31.40 (CDBUS2)
- net FTDI_UARTC_3V3_CTS: now reaches U31.41 (CDBUS3)
- net FTDI_UARTD_3V3_TXD: now reaches U31.48 (DDBUS0)
- net FTDI_UARTD_3V3_TXD: now also U34.10 (2B1)
- net FTDI_UARTD_3V3_RXD: now reaches U31.52 (DDBUS1)
- net FTDI_UARTD_3V3_RXD: now also U34.9 (GND)
- net FTDI_UARTD_3V3_RTC: now reaches U31.53 (DDBUS2)
- net FTDI_UARTD_3V3_CTS: now reaches U31.54 (DDBUS3)
- net at U31.6 (REF): now also C170.2, R70.1
- net at U31.7 (DM): now also U22.C3 (CH2_OUT+)
- net at U31.8 (DP): now also U22.C4 (CH2_OUT-)
- new net: C157.1, C158.1, U34.14 (VCCA)
- new net: C157.2, R68.1, U34.7 (1~{OE})
- new net: J23.A7 (D-), J23.B7 (D-), U22.A3 (CH2_IN+)
- new net: J23.A6 (D+), J23.B6 (D+), U22.A4 (CH2_IN-)
- new net: U33.10 (GND2), U33.15 (GND2), U33.9 (GND2)
- new net: U33.11 (VDD2), U33.16 (VDD2)
- new net: U33.2 (GND1), U33.7 (GND1), U33.8 (GND1)
- new net: C159.1, C160.1, C161.1, C162.1, C163.1, C164.1, C165.1, C166.1, C167.1, C168.1, C169.1
- new net: C140.1, C141.1, U32.14 (VCCA)
- new net: C140.2, R46.1, U32.7 (1~{OE})
- new net: J23.A1 (GND), J23.A12 (GND), J23.B1 (GND), J23.B12 (GND)
- new net: J23.A4 (VBUS), J23.A9 (VBUS), J23.B4 (VBUS), J23.B9 (VBUS)
- new net 3v3: C170.1
- no-connect marks 0 -> 24
Other:
- moved on the sheet: U31

Commit message: reorganization of the componentes
Parts:
- removed C139, C161, C162, C167: 100nF, Capacitor_SMD:C_0402_1005Metric, symbol Device:C_Small
- removed C168, C169: 1nF, Capacitor_SMD:C_0402_1005Metric, symbol Device:C_Small
- removed U33: TJA1052i-1, Package_SO:SOIC-16W_7.5x10.3mm_P1.27mm, symbol Interface_CAN_LIN:TJA1052i-1
- added C171, C174, C181, C182, C183, C184, C186: 100nF, Capacitor_SMD:C_0402_1005Metric, symbol Device:C_Small
- added C172, C173: 12Pf, Capacitor_SMD:C_0402_1005Metric, symbol Device:C_Small
- added C185: 10uF, Capacitor_SMD:C_0402_1005Metric, symbol Device:C_Small
- added L5, L6: 120R@10MHz, Inductor_SMD:L_0805_2012Metric, symbol Device:L_Ferrite
- added R71: 1M, Resistor_SMD:R_0402_1005Metric, symbol Device:R_Small
- added R72, R73: 150, Resistor_SMD:R_0402_1005Metric, symbol Device:R_Small
- added R74, R75, R76: 10k, Resistor_SMD:R_0402_1005Metric, symbol Device:R_Small
- added R77, R78: 5.1k, Resistor_SMD:R_0402_1005Metric, symbol Device:R_Small
- added U35: 93LCxxB, Package_DFN_QFN:DFN-8-1EP_3x2mm_P0.5mm_EP1.7x1.4mm, symbol Memory_EEPROM:93LCxxB
- added Y3: 12MHz, Crystal:Crystal_SMD_0603-4Pin_6.0x3.5mm, symbol Device:Crystal_GND24_Small
- C170: value 10uF -> 100nF
- J23: footprint (none) -> Connector_USB:USB_C_Receptacle_GCT_USB4110
- U32, U34: footprint (none) -> Package_DFN_QFN:UQFN-16_1.8x2.6mm_P0.4mm
Connections:
- net 3v3: now also R70.1, U31.50 (VREGIN), C171.1, C174.1, R74.1, R75.1, R76.1, U35.8 (VCC); no longer C170.1
- net GND: now also C170.2, U31.13 (TEST), C171.2, C172.2, C173.2, C174.2, C181.2, C182.2, C183.2, C184.2, C185.2, C186.2, R77.1, R78.1, U35.5 (GND), Y3.2, Y3.4; no longer R70.2
- net at C163.1, C164.1, C165.1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: now also U31.20 (VCCIO), U31.31 (VCCIO), U31.42 (VCCIO), U31.56 (VCCIO); no longer C159.1, C160.1
- net at J23.A5 (CC1): now also R78.2
- net at J23.B5 (CC2): now also R77.2
- net 1v8_VREGOUT: now reaches U31.12 (VCORE), U31.37 (VCORE), U31.64 (VCORE)
- net 1v8_VREGOUT: now also U31.49 (VREGOUT), C181.1, C182.1, C183.1, C184.1
- net at U31.2 (OSCI): now also C172.1, R71.1, Y3.1
- net at U31.3 (OSCO): now also R72.2
- net VPHY: now reaches U31.4 (VPHY)
- net VPHY: now also C185.1, C186.1, L5.2; no longer U31.9 (VPLL)
- net EEDATA: now reaches U31.61 (EEDATA)
- net EEDATA: now also R73.2, U35.3 (DI)
- net EECLK: now reaches U31.62 (EECLK)
- net EECLK: now also R74.2, U35.2 (SCLK)
- net EECS: now reaches U31.63 (EECS)
- net EECS: now also R76.2, U35.1 (CS)
- new net: R73.1, R75.2, U35.4 (DO)
- new net: C173.1, R71.2, R72.1, Y3.3
- new net: C170.1, R70.2, U31.6 (REF)
- new net VPLL: C159.1, C160.1, L6.2, U31.9 (VPLL)
- no-connect marks 24 -> 25
Other:
- moved on the sheet: C163, C164, C165, C166, C170, R70, U22B

Commit message: [PROCESSOR] Create zones It added power zones in the four layer
Changed lines of the file:
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@@
 		)
 	)
+	(global_label "jtag_Tx"
+		(shape input)
+		(at 185.42 52.07 0)
+		(fields_autoplaced yes)
+		(effects
+			(font
+				(size 1 1)
+			)
+			(justify left)
+		)
+		(property "Intersheetrefs" "${INTERSHEET_REFS}"
+			(at 192.9608 52.07 0)
+			(effects
+				(font
+					(size 1.27 1.27)
+				)
+				(justify left)
+				(hide yes)
+			)
+		)
+	)
+	(global_label "jtag_Rx"
+		(shape input)
+		(at 185.42 49.53 0)
+		(fields_autoplaced yes)
+		(effects
+			(font
+				(size 1 1)
+			)
+			(justify left)
+		)
+		(property "Intersheetrefs" "${INTERSHEET_REFS}"
+			(at 193.1989 49.53 0)
+			(effects
+				(font
+					(size 1.27 1.27)
+				)
+				(justify left)
+				(hide yes)
+			)
+		)
+	)
 	(symbol
 		(lib_id "power:GND")
@@
 	)
 	(symbol
-		(lib_name "_W_MX8M:SN74AVC4T774RSVR")
 		(lib_id "_W_MX8M:SN74AVC4T774RSVR")
 		(at 234.95 106.68 0)

Commit message: [BB_IMX8MLP IMX8MLP] Actuallizated to 9.0 kicad version
Parts:
- added J30: MCU-Serial, Connector_PinHeader_2.54mm:PinHeader_2x04_P2.54mm_Vertical, symbol Connector_Generic:Conn_02x04_Odd_Even
- C141, C158, C160, C163, C164, C165, C166, C170, C171, C174, C181, C182, C183, C184, C186: MP (none) -> C0402C104K4RACTU; Price (none) -> 0.1
- C172, C173: MP (none) -> C0402C120D5GACTU; Price (none) -> 0.5
- L5, L6: footprint Inductor_SMD:L_0805_2012Metric -> Inductor_SMD:L_0402_1005Metric
- R46, R68, R70, R74, R75, R76: MP (none) -> RC0402JR-0710KL; Price (none) -> 0.1
- R69: MP (none) -> RC0402FR-0712KL; Price (none) -> 0.1
- R71: MP (none) -> CRGCQ0402J1M0; Price (none) -> 0.1
- R72, R73: MP (none) -> CRCW0402150RFKEDC; Price (none) -> 0.1
- R77, R78: MP (none) -> RC0603FR-075K1L; Price (none) -> 0.1
- U22: MP (none) -> PCMF3USB3SZ; Price (none) -> 1.5
- U31: MP (none) -> FT4232H-56Q-TRAY; Price (none) -> 6.5
- U32, U34: value ~ -> SN74AVC4T774RSVR; MP (none) -> SN74AVC4T774RSVR; Price (none) -> 2
- U35: MP (none) -> 93LC46BT-I/MC; Price (none) -> 1
Connections:
- net FTDI_UARTC_3V3_RXD: now also J30.4 (Pin_4); no longer U34.11 (1B2)
- net FTDI_UARTC_3V3_TXD: now also J30.2 (Pin_2); no longer U34.12 (1B1)
- net FTDI_UARTD_3V3_RXD: now also J30.8 (Pin_8); no longer U34.9 (GND)
- net FTDI_UARTD_3V3_TXD: now also J30.6 (Pin_6); no longer U34.10 (2B1)
- net GND: no longer U32.9 (GND), U34.9 (GND)
- net JTAG_TCK: now reaches U32.1 (1A1)
- net JTAG_TDI: now reaches U32.2 (1A2)
- net JTAG_TDO: now reaches U32.3 (2A1)
- net JTAG_TMS: now reaches U32.4 (2A2)
- net at C170.1, R70.2: now also U31.14 (~{RESET}); no longer U31.6 (REF)
- net at R69.1: now also U31.6 (REF); no longer U31.14 (~{RESET})
- net UART2_TXD: now reaches U34.1 (1A1)
- net UART2_RXD: now reaches U34.2 (1A2)
- net UART4_TXD: now reaches U34.3 (2A1)
- net UART4_RXD: now reaches U34.4 (2A2)
- net mcu_UARTA_3V3_RXD renamed Serial_Rx
- net mcu_UARTA_3V3_TXD renamed Serial_Tx
- new net: J30.1 (Pin_1), U34.12 (1B1)
- new net: J30.3 (Pin_3), U34.11 (1B2)
- new net: J30.5 (Pin_5), U34.10 (2B1)
- new net: J30.7 (Pin_7), U34.9 (2B2)
Other:
- note added: "change footprint PCMF3USB1S MP PCMF1USB3SZ PR 0.5"
- moved on the sheet: C157, C158, R68, U34

Commit message: [LoRa] Starting a new project
Starting a new project base on LoRa LR1121, this project use
the module LBAA0XV2GT-001 that had sub-GHz and 2.4GHz frequencies.
Parts:
- removed U22: PCMF3USB3S, Package_CSP:Nexperia_WLCSP-15_6-3-6_2.37x1.17mm_Layout6x3_P0.4mm, symbol Power_Protection:PCMF3USB3S
- added U22: PCMF1USB3SZ, _W_SBC:BGA5N35P3X2_109X74X40N, symbol _W_MX8M:PCMF1HDMI2S
- L5, L6: footprint Inductor_SMD:L_0402_1005Metric -> _W_SBC:FIL_EXC-14CH120U; MP (none) -> EXC-14CE121U; Price (none) -> 0.3
- Y3: footprint Crystal:Crystal_SMD_0603-4Pin_6.0x3.5mm -> Crystal:Crystal_SMD_3225-4Pin_3.2x2.5mm; MP (none) -> ECS-120-8-33-JGN-TR; Price (none) -> 0.5
Connections:
- net GND: now also U32.15 (1DIR), U32.16 (2DIR), U32.6 (4DIR), U22.B1 (GND_CH1)
- net at J23.A7 (D-), J23.B7 (D-): now also U22.A1 (CH1_IN+)
- net at J23.A6 (D+), J23.B6 (D+): now also U22.A2 (CH1_IN-)
- net at U31.7 (DM): now also U22.C1 (CH1_OUT+)
- net at U31.8 (DP): now also U22.C2 (CH1_OUT-)
Other:
- note removed: "change footprint PCMF3USB1S MP PCMF1USB3SZ PR 0.5"
