File: Design_IMX8ML_Plus/IMX8ML_plus/storage.kicad_sch (KiCad schematic)
At the start: 24 parts, among them U1 MIMX8ML8CVNKZAB, U4 SDINBDG4-8G, U5 MT25QUxxxxxx1xW7, Y2 32.768KHz

Commit message: [IMX8ML] Add new layer
A new layers was add in the cpu schematic, now it had 8 layer.
Parts:
- added C159, C160: 2200pF, Capacitor_SMD:C_0201_0603Metric, symbol Device:C_Small
- added C161: 18pF, Capacitor_SMD:C_0201_0603Metric, symbol Device:C_Small
- added D2: LED, LED_SMD:LED_0603_1608Metric, symbol Device:LED
- added Q1: NX3008NBKW,115, Package_TO_SOT_SMD:SOT-323_SC-70, symbol Transistor_FET:2N7002
- added R42: 0, Resistor_SMD:R_0402_1005Metric, symbol Device:R_Small
- added R43: 550, Resistor_SMD:R_0402_1005Metric, symbol Device:R_Small
Connections:
- net GND: now also C159.2, C160.2, C161.2, Q1.2 (S)
- net MIPI_VREG1_CAP: now reaches U1.F18 (MIPI_VREG1_CAP)
- net MIPI_VREG1_CAP: now also C160.1
- net MIPI_TEST_DNU: now reaches U1.F24 (MIPI_TEST_DNU)
- net MIPI_TEST_DNU: now also C159.1
- net NAND_DQS: now reaches U1.R26 (NAND_DQS)
- net NAND_DQS: now also C161.1, R42.2
- net NAND_READY_B: now reaches U1.T28 (NAND_READY_B)
- net NAND_READY_B: now also Q1.1 (G)
- net PMIC_RST_B renamed PMIC_STBY_REC
- new net: D2.1 (K), Q1.3 (D)
- new net: D2.2 (A), R43.2
- new net +3V3: R43.1
- new net NAND_DQS_PINOUT: R42.1
Other:
- note added: "ON/OFF[G22] PinOUT(BUTTON) POR_B [J29] PMIC PMIC_ON_REQ [F22] PMI PMIC_STBY_REQ [J24] PMIC"
- note added: "SAI1_TXFS ETH_2_RGMII_RX_CTL SAI1_TXC ETH_2_RGMII_RXC"
- note removed: "ETH_2_RGMII_RXC"
- note removed: "ETH_2_RGMII_RX_CTL"
